File: pcb_design/pcb_design.kicad_sch (KiCad schematic)
At the start: 35 parts, among them J1 USB_C_Receptacle_USB2.0_16P, J2 Conn_01x02_Pin, J3 Conn_01x02_Pin, J4 Conn_01x02_Pin, Q1 MMBT3904, Q2 MMBT3904, U1 AP2112K-3.3, U2 ESP32-C3-WROOM-02, U3 MPU-6050, U4 QMC6308, U5 AP2112K-1.8, U6 TXS0102DCU, U7 MCP73831-2-OT

Commit message: feat: implement interruptor to turn on or off the 'acpi_pulsera'
Parts:
- added R10: 1M, Resistor_SMD:R_0603_1608Metric, symbol Device:R
- added SW1: SW_SPDT, Button_Switch_SMD:SW_SPDT_Shouhan_MSK12C02, symbol Switch:SW_SPDT
Connections:
- net GND: now also SW1.1 (A)
- net VBAT: now also R10.2; no longer U1.3 (EN)
- new net: R10.1, SW1.2 (B), U1.3 (EN)
- no-connect marks 15 -> 16
Changed lines of the file:
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@@
 	)
 	(junction
-		(at 115.57 26.67)
-		(diameter 0)
-		(color 0 0 0 0)
-	)
-	(junction
 		(at 154.94 134.62)
 		(diameter 0)
@@
 	)
 	(junction
+		(at 148.59 39.37)
+		(diameter 0)
+		(color 0 0 0 0)
+	)
+	(junction
 		(at 62.23 151.13)
 		(diameter 0)
@@
 		(color 0 0 0 0)
 	)
+	(junction
+		(at 100.33 26.67)
+		(diameter 0)
+		(color 0 0 0 0)
+	)
+	(junction
+		(at 118.11 41.91)
+		(diameter 0)
+		(color 0 0 0 0)
+	)
 	(no_connect
 		(at 204.47 109.22)
@@
 	)
 	(no_connect
+		(at 143.51 59.69)
+	)
+	(no_connect
 		(at 173.99 129.54)
 	)
@@
 	(wire
 		(pts
+			(xy 100.33 49.53) (xy 100.33 26.67)
+		)
+		(stroke
+			(width 0)
+			(type default)
+		)
+	)
+	(wire
+		(pts
 			(xy 62.23 151.13) (xy 62.23 156.21)
 		)
@@
 	(wire
 		(pts
+			(xy 133.35 41.91) (xy 118.11 41.91)
+		)
+		(stroke
+			(width 0)
+			(type default)
+		)
+	)
+	(wire
+		(pts
 			(xy 82.55 157.48) (xy 82.55 161.29)
 		)
@@
 	(wire
 		(pts
-			(xy 118.11 166.37) (xy 118.11 173.99)
+			(xy 118.11 49.53) (xy 100.33 49.53)
 		)
 		(stroke
@@
 	(wire
 		(pts
-			(xy 162.56 83.82) (xy 162.56 116.84)
+			(xy 118.11 166.37) (xy 118.11 173.99)
 		)
 		(stroke
@@
 	(wire
 		(pts
-			(xy 90.17 151.13) (xy 90.17 148.59)
+			(xy 162.56 83.82) (xy 162.56 116.84)
 		)
 		(stroke
@@
 	(wire
 		(pts
-			(xy 110.49 85.09) (xy 110.49 153.67)
+			(xy 90.17 151.13) (xy 90.17 148.59)
 		)
 		(stroke
@@
 	(wire
 		(pts
-			(xy 118.11 29.21) (xy 115.57 29.21)
+			(xy 110.49 85.09) (xy 110.49 153.67)
 		)
 		(stroke
@@
 	(wire
 		(pts
+			(xy 118.11 29.21) (xy 118.11 41.91)
+		)
+		(stroke
+			(width 0)
+			(type default)
+		)
+	)
+	(wire
+		(pts
 			(xy 148.59 97.79) (xy 148.59 101.6)
 		)
@@
 	(wire
 		(pts
+			(xy 148.59 39.37) (xy 156.21 39.37)
+		)
+		(stroke
+			(width 0)
+			(type default)
+		)
+	)
+	(wire
+		(pts
 			(xy 242.57 109.22) (xy 254 109.22)
 		)
@@
 	(wire
 		(pts
-			(xy 81.28 86.36) (xy 85.09 86.36)
+			(xy 148.59 54.61) (xy 148.59 39.37)
 		)
 		(stroke
@@
 	(wire
 		(pts
-			(xy 115.57 26.67) (xy 118.11 26.67)
+			(xy 81.28 86.36) (xy 85.09 86.36)
 		)
 		(stroke
@@
 	(wire
 		(pts
-			(xy 115.57 29.21) (xy 115.57 26.67)
-		)
-		(stroke
-			(width 0)
-			(type default)
-		)
-	)
-	(wire
-		(pts
 			(xy 143.51 39.37) (xy 143.51 43.18)
 		)
@@
 	(wire
 		(pts
-			(xy 143.51 39.37) (xy 156.21 39.37)
+			(xy 143.51 39.37) (xy 148.59 39.37)
 		)
 		(stroke
@@
 	(wire
 		(pts
-			(xy 85.09 26.67) (xy 115.57 26.67)
+			(xy 85.09 26.67) (xy 100.33 26.67)
 		)
 		(stroke
@@
 	(wire
 		(pts
+			(xy 100.33 26.67) (xy 118.11 26.67)
+		)
+		(stroke
+			(width 0)
+			(type default)
+		)
+	)
+	(wire
+		(pts
 			(xy 156.21 34.29) (xy 156.21 39.37)
 		)
@@
 	(wire
 		(pts
+			(xy 143.51 54.61) (xy 148.59 54.61)
+		)
+		(stroke
+			(width 0)
+			(type default)
+		)
+	)
+	(wire
+		(pts
 			(xy 58.42 63.5) (xy 58.42 71.12)
 		)
@@
 	(wire
 		(pts
+			(xy 133.35 57.15) (xy 133.35 41.91)
+		)
+		(stroke
+			(width 0)
+			(type default)
+		)
+	)
+	(wire
+		(pts
 			(xy 86.36 154.94) (xy 86.36 168.91)
 		)
@@
 	)
 	(symbol
+		(lib_id "Device:R")
+		(at 118.11 45.72 0)
+		(unit 1)
+		(body_style 1)
+		(exclude_from_sim no)
+		(in_bom yes)
+		(on_board yes)
+		(in_pos_files yes)
+		(dnp no)
+		(fields_autoplaced yes)
+		(property "Reference" "R10"
+			(at 120.65 44.4499 0)
+			(show_name no)
+			(do_not_autoplace no)
+			(effects
+				(font
+					(size 1.27 1.27)
+				)
+				(justify left)
+			)
+		)
+		(property "Value" "1M"
+			(at 120.65 46.9899 0)
+			(show_name no)
+			(do_not_autoplace no)
+			(effects
+				(font
+					(size 1.27 1.27)
+				)
+				(justify left)
+			)
+		)
+		(property "Footprint" "Resistor_SMD:R_0603_1608Metric"
+			(at 116.332 45.72 90)
+			(hide yes)
+			(show_name no)
+			(do_not_autoplace no)
+			(effects
+				(font
+					(size 1.27 1.27)
+				)
+			)
+		)
+		(property "Datasheet" ""
+			(at 118.11 45.72 0)
+			(hide yes)
+			(show_name no)
+			(do_not_autoplace no)
+			(effects
+				(font
+					(size 1.27 1.27)
+				)
+			)
+		)
+		(property "Description" "Resistor"
+			(at 118.11 45.72 0)
+			(hide yes)
+			(show_name no)
+			(do_not_autoplace no)
+			(effects
+				(font
+					(size 1.27 1.27)
+				)
+			)
+		)
+		(pin "1"
+		)
+		(pin "2"
+		)
+		(instances
+			(project "pcb_design"
+				(path "/ed89a1db-d160-432e-90bf-e0dcbc334e75"
+					(reference "R10")
+					(unit 1)
+				)
+			)
+		)
+	)
+	(symbol
 		(lib_id "Connector:Conn_01x02_Pin")
 		(at 254 90.17 90)
@@
 					(unit 1)
 				)
+			)
+		)
+	)
+	(symbol
+		(lib_id "Switch:SW_SPDT")
+		(at 138.43 57.15 0)
+		(unit 1)
+		(body_style 1)
+		(exclude_from_sim no)
+		(in_bom yes)
+		(on_board yes)
+		(in_pos_files yes)
+		(dnp no)
+		(fields_autoplaced yes)
+		(property "Reference" "SW1"
+			(at 138.43 48.26 0)
+			(show_name no)
+			(do_not_autoplace no)
+			(effects
+				(font
+					(size 1.27 1.27)
+				)
+			)
+		)
+		(property "Value" "SW_SPDT"
+			(at 138.43 50.8 0)
+			(show_name no)
+			(do_not_autoplace no)
+			(effects
+				(font
+					(size 1.27 1.27)
+				)
+			)
+		)
+		(property "Footprint" "Button_Switch_SMD:SW_SPDT_Shouhan_MSK12C02"
+			(at 138.43 57.15 0)
+			(hide yes)
+			(show_name no)
+			(do_not_autoplace no)
+			(effects
+				(font
+					(size 1.27 1.27)
+				)
+			)
+		)
+		(property "Datasheet" ""
+			(at 138.43 64.77 0)
+			(hide yes)
+			(show_name no)
+			(do_not_autoplace no)
+			(effects
+				(font
+					(size 1.27 1.27)
+				)
+			)
+		)
+		(property "Description" "Switch, single pole double throw"
+			(at 138.43 57.15 0)
+			(hide yes)
+			(show_name no)
+			(do_not_autoplace no)
+			(effects
+				(font
+					(size 1.27 1.27)
+				)
+			)
+		)
+		(pin "2"
+		)
+		(pin "3"
+		)
+		(pin "1"
+		)
+		(instances
+			(project "pcb_design"
+				(path "/ed89a1db-d160-432e-90bf-e0dcbc334e75"
+					(reference "SW1")
+					(unit 1)
+				)

Commit message: feat: implement correct footprint of JST connectors
Parts:
- J2, J3: value Conn_01x02_Pin -> JST_PH_S2B-PH-K; footprint Connector_PinHeader_2.54mm:PinHeader_1x02_P2.54mm_Vertical -> Connector_JST:JST_PH_S2B-PH-K_1x02_P2.00mm_Horizontal
- J4: value Conn_01x02_Pin -> JST_PH_S2B-PH-K; footprint (none) -> Connector_JST:JST_PH_S2B-PH-K_1x02_P2.00mm_Horizontal
Changed lines of the file:
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@@
 			)
 		)
-		(property "Value" "Conn_01x02_Pin"
+		(property "Value" "JST_PH_S2B-PH-K"
 			(at 257.81 118.7449 90)
 			(show_name no)
@@
 			)
 		)
-		(property "Footprint" "Connector_PinHeader_2.54mm:PinHeader_1x02_P2.54mm_Vertical"
+		(property "Footprint" "Connector_JST:JST_PH_S2B-PH-K_1x02_P2.00mm_Horizontal"
 			(at 254 118.11 0)
 			(hide yes)
@@
 			)
 		)
-		(property "Value" "Conn_01x02_Pin"
+		(property "Value" "JST_PH_S2B-PH-K"
 			(at 257.81 90.8049 90)
 			(show_name no)
@@
 			)
 		)
-		(property "Footprint" "Connector_PinHeader_2.54mm:PinHeader_1x02_P2.54mm_Vertical"
+		(property "Footprint" "Connector_JST:JST_PH_S2B-PH-K_1x02_P2.00mm_Horizontal"
 			(at 254 90.17 0)
 			(hide yes)
@@
 			)
 		)
-		(property "Value" "Conn_01x02_Pin"
+		(property "Value" "JST_PH_S2B-PH-K"
 			(at 39.37 23.4949 90)
 			(show_name no)
@@
 			)
 		)
-		(property "Footprint" ""
+		(property "Footprint" "Connector_JST:JST_PH_S2B-PH-K_1x02_P2.00mm_Horizontal"
 			(at 38.1 21.59 0)
 			(hide yes)

Commit message: feat: implement complete pcb design
Parts:
- D1, D2: value 1N4148 -> 1N4148W; footprint Diode_THT:D_DO-35_SOD27_P7.62mm_Horizontal -> Diode_SMD:D_SOD-123; LCSC Part (none) -> C81598
- J1: LCSC Part (none) -> C165948
- J2, J3, J4: LCSC Part (none) -> C265016
- Q1, Q2: LCSC Part (none) -> C20526
- SW1: LCSC Part (none) -> C431540
- U1: LCSC Part (none) -> C51118
- U2: LCSC Part (none) -> C2934560
- U3: LCSC Part (none) -> C24112
- U5: LCSC Part (none) -> C176944
- U6: LCSC Part (none) -> C53434
- U7: LCSC Part (none) -> C424093
Changed lines of the file:
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@@
 			)
 		)
+		(property "LCSC Part" "C24112"
+			(at 130.81 102.87 0)
+			(hide yes)
+			(show_name no)
+			(do_not_autoplace no)
+			(effects
+				(font
+					(size 1.27 1.27)
+				)
+			)
+		)
 		(pin "4"
 		)
@@
 			)
 		)
+		(property "LCSC Part" "C2934560"
+			(at 189.23 126.365 0)
+			(hide yes)
+			(show_name no)
+			(do_not_autoplace no)
+			(effects
+				(font
+					(size 1.27 1.27)
+				)
+			)
+		)
 		(pin "17"
 		)
@@
 			)
 		)
-		(property "Value" "1N4148"
+		(property "Value" "1N4148W"
 			(at 245.11 80.0099 90)
 			(show_name no)
@@
 			)
 		)
-		(property "Footprint" "Diode_THT:D_DO-35_SOD27_P7.62mm_Horizontal"
+		(property "Footprint" "Diode_SMD:D_SOD-123"
 			(at 242.57 78.74 0)
 			(hide yes)
@@
 			)
 		)
-		(property "Description" "100V 0.15A standard switching diode, DO-35"
+		(property "Description" "100V 0.15A standard switching diode, SOD-123 SMD"
+			(at 242.57 78.74 0)
+			(hide yes)
+			(show_name no)
+			(do_not_autoplace no)
+			(effects
+				(font
+					(size 1.27 1.27)
+				)
+			)
+		)
+		(property "LCSC Part" "C81598"
 			(at 242.57 78.74 0)
 			(hide yes)
@@
 			)
 		)
+		(property "LCSC Part" "C265016"
+			(at 254 118.11 0)
+			(hide yes)
+			(show_name no)
+			(do_not_autoplace no)
+			(effects
+				(font
+					(size 1.27 1.27)
+				)
+			)
+		)
 		(pin "1"
 		)
@@
 			)
 		)
+		(property "LCSC Part" "C51118"
+			(at 125.73 29.21 0)
+			(hide yes)
+			(show_name no)
+			(do_not_autoplace no)
+			(effects
+				(font
+					(size 1.27 1.27)
+				)
+			)
+		)
 		(pin "1"
 		)
@@
 			)
 		)
+		(property "LCSC Part" "C424093"
+			(at 27.94 106.68 0)
+			(hide yes)
+			(show_name no)
+			(do_not_autoplace no)
+			(effects
+				(font
+					(size 1.27 1.27)
+				)
+			)
+		)
 		(pin "2"
 		)
@@
 			)
 		)
+		(property "LCSC Part" "C265016"
+			(at 254 90.17 0)
+			(hide yes)
+			(show_name no)
+			(do_not_autoplace no)
+			(effects
+				(font
+					(size 1.27 1.27)
+				)
+			)
+		)
 		(pin "1"
 		)
@@
 			)
 		)
+		(property "LCSC Part" "C53434"
+			(at 72.39 163.83 0)
+			(hide yes)
+			(show_name no)
+			(do_not_autoplace no)
+			(effects
+				(font
+					(size 1.27 1.27)
+				)
+			)
+		)
 		(pin "7"
 		)
@@
 			)
 		)
+		(property "LCSC Part" "C176944"
+			(at 73.66 123.19 0)
+			(hide yes)
+			(show_name no)
+			(do_not_autoplace no)
+			(effects
+				(font
+					(size 1.27 1.27)
+				)
+			)
+		)
 		(pin "4"
 		)
@@
 			)
 		)
+		(property "LCSC Part" "C431540"
+			(at 138.43 57.15 0)
+			(hide yes)
+			(show_name no)
+			(do_not_autoplace no)
+			(effects
+				(font
+					(size 1.27 1.27)
+				)
+			)
+		)
 		(pin "2"
 		)
@@
 			)
 		)
+		(property "LCSC Part" "C265016"
+			(at 38.1 21.59 0)
+			(hide yes)
+			(show_name no)
+			(do_not_autoplace no)
+			(effects
+				(font
+					(size 1.27 1.27)
+				)
+			)
+		)
 		(pin "1"
 		)
@@
 			)
 		)
-		(property "Value" "1N4148"
+		(property "Value" "1N4148W"
 			(at 245.11 106.6799 90)
 			(show_name no)
@@
 			)
 		)
-		(property "Footprint" "Diode_THT:D_DO-35_SOD27_P7.62mm_Horizontal"
+		(property "Footprint" "Diode_SMD:D_SOD-123"
 			(at 242.57 105.41 0)
 			(hide yes)
@@
 			)
 		)
-		(property "Description" "100V 0.15A standard switching diode, DO-35"
+		(property "Description" "100V 0.15A standard switching diode, SOD-123 SMD"
+			(at 242.57 105.41 0)
+			(hide yes)
+			(show_name no)
+			(do_not_autoplace no)
+			(effects
+				(font
+					(size 1.27 1.27)
+				)
+			)
+		)
+		(property "LCSC Part" "C81598"
 			(at 242.57 105.41 0)
 			(hide yes)
@@
 			)
 		)
+		(property "LCSC Part" "C20526"
+			(at 224.79 83.82 0)
+			(hide yes)
+			(show_name no)
+			(do_not_autoplace no)
+			(effects
+				(font
+					(size 1.27 1.27)
+				)
+			)
+		)
 		(property "Sim.Device" "NPN"
 			(at 224.79 83.82 0)
@@
 			)
 		)
+		(property "LCSC Part" "C20526"
+			(at 224.79 106.68 0)
+			(hide yes)
+			(show_name no)
+			(do_not_autoplace no)
+			(effects
+				(font
+					(size 1.27 1.27)
+				)
+			)
+		)
 		(property "Sim.Device" "NPN"
 			(at 224.79 106.68 0)
@@
 			(at 58.42 86.36 0)
 			(hide yes)
+			(show_name no)
+			(do_not_autoplace no)
+			(effects
+				(font
+					(size 1.27 1.27)
+				)
+			)
+		)
+		(property "LCSC Part" "C165948"
+			(at 58.42 86.36 0)
+			(hide yes)
